File: p2.sch (KiCad schematic (older format))
At the start: 25 parts, among them J1 BARREL_JACK, J2 FLASH_JMP, J3 UART, J4 ALT_POWER, J5 jack-3.5mm-5pin, J6 jack-3.5mm-5pin, J7 jack-3.5mm-5pin, J8 jack-3.5mm-5pin, Q1 IRL540N, Q2 IRL540N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

Commit message: update to pcb-rev1.1
Parts:
- Q2: footprint TO_SOT_Packages_THT:TO-220_Horizontal -> TO_SOT_Packages_THT:TO-220_Horizontal_Reversed
- U2: value ESP-12E -> ESP-12F
Changed lines of the file:
@@
 Title "P2 - WaterControl v2"
 Date "2017-04-24"
-Rev "3.3"
+Rev "3.4"
 Comp "mr"
 Comment1 ""
@@
 P 5350 3750
 F 0 "U2" H 5350 3650 50  0000 C CNN
-F 1 "ESP-12E" H 5350 3850 50  0000 C CNN
+F 1 "ESP-12F" H 5350 3850 50  0000 C CNN
 F 2 "esp8266:ESP-12E" H 5350 3750 50  0001 C CNN
 F 3 "" H 5350 3750 50  0001 C CNN
@@
 F 0 "Q2" H 8750 5375 50  0000 L CNN
 F 1 "IRL540N" H 8750 5300 50  0000 L CNN
-F 2 "TO_SOT_Packages_THT:TO-220_Horizontal" H 8750 5225 50  0001 L CIN
+F 2 "TO_SOT_Packages_THT:TO-220_Horizontal_Reversed" H 8750 5225 50  0001 L CIN
 F 3 "" H 8500 5300 50  0001 L CNN
 	1    8500 5300

Commit message: current state sync
Parts:
- removed C1: 10uF, Capacitors_THT:CP_Radial_Tantal_D5.0mm_P2.50mm, symbol CP
- removed R1, R2, R6, R7: 10k, Resistors_THT:R_Axial_DIN0207_L6.3mm_D2.5mm_P7.62mm_Horizontal, symbol R
- removed U1: LM1117IMP-33, TO_SOT_Packages_SMD:SOT-223, symbol LM1117IMP-33
- removed U2: ESP-12F, esp8266:ESP-12E, symbol ESP-12E
- added LED1, LED2: LED, LEDs:LED_D3.0mm_Horizontal_O1.27mm_Z2.0mm, symbol LED
- added R8, R9: 1k, Resistors_THT:R_Axial_DIN0207_L6.3mm_D2.5mm_P7.62mm_Horizontal, symbol R
- added RN1: 10k, Resistors_THT:R_Array_SIP5, symbol R_Network04
- added U1: R-78E3.3-0.5, myfootprints:DCDC-Conv_Recom_R-78Exx-0.5, symbol R-78E3.3-0.5
- added U2: ESP-12, esp8266:ESP-12, symbol ESP-12
- added U3: Switch, Buttons_Switches_THT:SW_PUSH_6mm, symbol Switch
- C2: value 10uF -> 10u
- C3, C4: value 100nF -> 100n
- J4: value ALT_POWER -> ALT_Pwr
Connections:
- net labels added: +12V, +3.3V, led1, led2, pump1, pump2, wifi-sw
- net labels removed: HEAT_Vcc
- wire segments 45 -> 56
- no-connect marks 25 -> 16
Other:
- note added: "2 signal LEDs"
- note added: "Water Sensor Wiring (with Pullup-Resistor in the basic ESP wiring)"
- note added: "wifi-switch"
- note removed: "Water Sensor Wiring (with Pullup-Resistor)"

Commit message: rev4.1 - switched to capacitive sensors by including a multiplexer, added another switch, rotated both.
Parts:
- removed C2: 10u, Capacitors_THT:CP_Radial_Tantal_D5.0mm_P2.50mm, symbol CP
- removed C3, C4: 100n, Capacitors_THT:C_Disc_D5.0mm_W2.5mm_P5.00mm, symbol C
- removed D1, D2: 1N4002, Diodes_THT:D_A-405_P10.16mm_Horizontal, symbol D
- removed J1: BARREL_JACK, myfootprints:Barrel_Jack_5.5_2.1mm, symbol BARREL_JACK
- removed J2: FLASH_JMP, Pin_Headers:Pin_Header_Straight_1x03_Pitch2.54mm, symbol CONN_01X03
- removed J3: UART, Pin_Headers:Pin_Header_Straight_1x04_Pitch2.54mm, symbol CONN_01X04
- removed J4: ALT_Pwr, Pin_Headers:Pin_Header_Straight_1x02_Pitch2.54mm, symbol CONN_01X02
- removed J5, J6, J7, J8: jack-3.5mm-5pin, myfootprints:3.5mm_5pin_jack, symbol jack-3.5mm-5pin
- removed LED1, LED2: LED, LEDs:LED_D3.0mm_Horizontal_O1.27mm_Z2.0mm, symbol LED
- removed Q1: IRL540N, TO_SOT_Packages_THT:TO-220_Horizontal, symbol IRL540N
- removed Q2: IRL540N, TO_SOT_Packages_THT:TO-220_Horizontal_Reversed, symbol IRL540N
- removed R3: 10k, Resistors_THT:R_Axial_DIN0207_L6.3mm_D2.5mm_P7.62mm_Horizontal, symbol R
- removed R4, R5, R8, R9: 1k, Resistors_THT:R_Axial_DIN0207_L6.3mm_D2.5mm_P7.62mm_Horizontal, symbol R
- removed RN1: 10k, Resistors_THT:R_Array_SIP5, symbol R_Network04
- removed U1: R-78E3.3-0.5, myfootprints:DCDC-Conv_Recom_R-78Exx-0.5, symbol R-78E3.3-0.5
- removed U2: ESP-12, esp8266:ESP-12, symbol ESP-12
- removed U3: Switch, Buttons_Switches_THT:SW_PUSH_6mm, symbol Switch
- added C1, C2: 100n, Capacitor_THT:C_Disc_D5.0mm_W2.5mm_P5.00mm, symbol Device:C
- added C3: 10u, Capacitor_THT:CP_Radial_Tantal_D5.0mm_P2.50mm, symbol Device:CP
- added D1, D2: 1N4002, Diode_THT:D_A-405_P10.16mm_Horizontal, symbol Diode:1N4002
- added J1: FLASH_JMP, myfootprints:PinHeader_2.54mm_1x3_short, symbol Connector:Conn_01x03_Male
- added J2: UART, Connector_PinHeader_2.54mm:PinHeader_1x04_P2.54mm_Vertical, symbol Connector:Conn_01x04_Male
- added J3: ALT_Pwr, Connector_PinHeader_2.54mm:PinHeader_1x02_P2.54mm_Vertical, symbol Connector:Conn_01x02_Male
- added J4: BARREL_JACK, myfootprints:Barrel_Jack_5.5_2.1mm, symbol myschematics:BARREL_JACK
- added J5, J6, J7, J8: jack-3.5mm-5pin, myfootprints:3.5mm_5pin_jack, symbol myschematics:jack-3.5mm-5pin
- added LED1, LED2: LED, LED_THT:LED_D3.0mm_Horizontal_O1.27mm_Z2.0mm_Clear, symbol Device:LED
- added Q1: IRL540N, Package_TO_SOT_THT:TO-220-3_Horizontal_TabUp, symbol myschematics:IRL540N
- added Q2: IRL540N, Package_TO_SOT_THT:TO-220-3_Horizontal_TabDown, symbol myschematics:IRL540N
- added R1: 10k, Resistor_THT:R_Axial_DIN0207_L6.3mm_D2.5mm_P7.62mm_Horizontal, symbol Device:R
- added R5: 220k, Resistor_THT:R_Axial_DIN0207_L6.3mm_D2.5mm_P7.62mm_Horizontal, symbol Device:R
- added R6: 100k, Resistor_THT:R_Axial_DIN0207_L6.3mm_D2.5mm_P7.62mm_Horizontal, symbol Device:R
- added RN1: 1k, myfootprints:ResistorArrayx4-27185436, symbol Device:R_Pack04
- added RN2: 10k, myfootprints:ResistorArrayx4-18726345, symbol Device:R_Pack04
- added SW1, SW2: SW_Push, Button_Switch_THT:SW_Tactile_SPST_Angled_PTS645Vx58-2LFS, symbol Switch:SW_Push
- added U1: R-78E3.3-0.5, myfootprints:DCDC-Conv_Recom_R-78Exx-0.5, symbol Regulator_Switching:R-78E3.3-0.5
- added U2: ESP-12, ESP8266:ESP-12, symbol ESP8266:ESP-12
- added U3: 74LVC1G3157, Package_TO_SOT_SMD:SOT-363_SC-70-6_Handsoldering, symbol 74xGxx:74LVC1G3157
Connections:
- net labels added: 10k_to_3v3_1, 10k_to_3v3_2, 10k_to_gnd_1, 10k_to_gnd_2, GPIO_0_Flash, pump_ctl_1, pump_ctl_2, sensor_in, sensor_switch, sw_1, sw_2
- net labels removed: GPIO0, ctl1, ctl2, ctl3, ctl4, pump1, pump2, wifi-sw
- wire segments 56 -> 90
- no-connect marks 16 -> 13
Other:
- note added: "LEDs and switches"
- note added: "MCU"
- note added: "Pin-Headers"
- note added: "Power Supply and Voltage regulator"
- note added: "Pump connectors"
- note added: "Sensor Connectors"
- note added: "can be used for wakeup"
- note added: "must be down on boot"
- note added: "on-board led"
- note removed: "2 signal LEDs"
- note removed: "Alternative Power Supply Header (12VDC)"
- note removed: "Basic ESP-12F Wiring"
- note removed: "EnableFlashing-Jumper"
- note removed: "Power Supply and Voltage regulator (12V->3.3V)"
- note removed: "Pump Controls"
- note removed: "UART-Header"
- note removed: "Water Sensor Wiring (with Pullup-Resistor in the basic ESP wiring)"
- note removed: "wifi-switch"
